Commit message: namespace and prefix changes

File: ur5e_2f85_description/urdf/ur5e_2f85.xacro (robot description, xacro)
@@ -5,10 +5,10 @@
     <xacro:include filename="$(find robotiq_2f_85_gripper_visualization)/urdf/robotiq_arg2f_85_model_macro.xacro" />
     <!-- parameters -->
-    <xacro:arg name="ur5e_prefix" default="" />
+    <xacro:arg name="arm_prefix" default="" />
     <xacro:arg name="kinematics_params" default="$(find ur5e_2f85_description)/config/ur5e_kinematics_calib.yaml" />
     <xacro:arg name="gripper_prefix" default="" />
     <!-- instantiate robot and gripper macros -->
     <xacro:ur5e_robot
-      prefix="$(arg ur5e_prefix)"
+      prefix="$(arg arm_prefix)"
       kinematics_parameters_file="$(arg kinematics_params)"
     />
@@ -19,11 +19,11 @@
     <joint name="world_to_ur5e" type="fixed">
       <parent link="world" />
-      <child link = "$(arg ur5e_prefix)base_link" />
+      <child link = "$(arg arm_prefix)base_link" />
       <origin xyz="-0.0 0 0" rpy="0 0 0" />
     </joint>
     <!-- add gripper to robot -->
-    <joint name="$(arg ur5e_prefix)robotiq_arg2f_base_joint" type="fixed">
-      <origin xyz="0 0 0" rpy="0 0 0" />
-      <parent link="$(arg ur5e_prefix)tool0" />
+    <joint name="$(arg arm_prefix)robotiq_arg2f_base_joint" type="fixed">
+      <origin xyz="0 0 0" rpy="0 0 ${-pi/2}" />
+      <parent link="$(arg arm_prefix)tool0" />
       <child link="$(arg gripper_prefix)robotiq_arg2f_base_link"/>
     </joint>
