Commit message: created macro for robot arm with gripper

File: ur5e_2f85_description/urdf/ur5e_2f85.urdf.xacro (robot description, xacro)
@@ -1,30 +1,22 @@
 <?xml version="1.0"?>
 <robot xmlns:xacro="http://ros.org/wiki/xacro" name="ur5e_2f85_robot">
-    <!-- include robot and gripper xacro macros -->
-    <xacro:include filename="$(find ur5e_2f85_description)/urdf/ur5e_macro.xacro" />
-    <xacro:include filename="$(find robotiq_2f_85_gripper_visualization)/urdf/robotiq_arg2f_85_model_macro.xacro" />
-    <!-- parameters -->
-    <xacro:arg name="arm_prefix" default="" />
-    <xacro:arg name="kinematics_params" default="$(find ur5e_2f85_description)/config/ur5e_kinematics_calib.yaml" />
-    <xacro:arg name="gripper_prefix" default="" />
-    <!-- instantiate robot and gripper macros -->
-    <xacro:ur5e_robot
-      prefix="$(arg arm_prefix)"
-      kinematics_parameters_file="$(arg kinematics_params)"
-    />
-    <xacro:robotiq_arg2f_85
-      prefix="$(arg gripper_prefix)"
-    />
-    <link name="world"/>
-    <joint name="world_to_ur5e" type="fixed">
-      <parent link="world" />
-      <child link = "$(arg arm_prefix)base_link" />
-      <origin xyz="-0.0 0 0" rpy="0 0 0" />
-    </joint>
-    <!-- add gripper to robot -->
-    <joint name="$(arg arm_prefix)robotiq_arg2f_base_joint" type="fixed">
-      <origin xyz="0 0 0" rpy="0 0 ${-pi/2}" />
-      <parent link="$(arg arm_prefix)tool0" />
-      <child link="$(arg gripper_prefix)robotiq_arg2f_base_link"/>
-    </joint>
+  <!-- include robot with gripper xacro macro -->
+  <xacro:include filename="$(find ur5e_2f85_description)/urdf/ur5e_2f85_macro.xacro" />
+  <!-- parameters -->
+  <xacro:arg name="arm_prefix" default="" />
+  <xacro:arg name="kinematics_params" default="$(find ur5e_2f85_description)/config/ur5e_kinematics_calib.yaml" />
+  <xacro:arg name="gripper_prefix" default="" />
+  <!-- instantiate robot with gripper macro -->
+  <xacro:ur5e_2f85_robot
+    arm_prefix="$(arg arm_prefix)"
+    kinematics_parameters_file="$(arg kinematics_params)"
+    gripper_prefix="$(arg gripper_prefix)"
+  />
+  <!-- link robot to world -->
+  <link name="world"/>
+  <joint name="world_to_ur5e" type="fixed">
+    <parent link="world" />
+    <child link = "$(arg arm_prefix)base_link" />
+    <origin xyz="0 0 0" rpy="0 0 0" />
+  </joint>
 </robot>
