Commit message: renamed mobile colaborative arm package

File: moca_description/urdf/moca.urdf.xacro (robot description, xacro)
@@ -1,6 +1,6 @@
 <?xml version="1.0"?>
-<robot xmlns:xacro="http://ros.org/wiki/xacro" name="mia_robot">
+<robot xmlns:xacro="http://ros.org/wiki/xacro" name="moca_robot">
   <!-- include robot macro -->
-  <xacro:include filename="$(find mia_description)/urdf/mia_macro.xacro" />
+  <xacro:include filename="$(find moca_description)/urdf/moca_macro.xacro" />
   <!-- mir100 parameters -->
   <xacro:arg name="mir_type" default="mir_100" />
@@ -12,5 +12,5 @@
   <xacro:arg name="gripper_prefix" default="2f85_" />
   <!-- instantiate robot with gripper macro -->
-  <xacro:mia_robot
+  <xacro:moca_robot
     mir_prefix="$(arg mir_prefix)"
     arm_prefix="$(arg arm_prefix)"

File: moca_description/urdf/moca_macro.xacro (robot description, xacro)
@@ -1,5 +1,5 @@
 <?xml version="1.0"?>
 <robot xmlns:xacro="http://ros.org/wiki/xacro">
-  <xacro:macro name="mia_robot" params="
+  <xacro:macro name="moca_robot" params="
     mir_prefix
     arm_prefix
