Commit message: corrected moca enclosure dimensions and arm origin

File: moca_description/urdf/moca_macro.xacro (robot description, xacro)
@@ -36,7 +36,7 @@
     <link name="enclosure">
         <visual>
-            <origin xyz="0 0 0.2" rpy="0 0 0"/>
+            <origin xyz="0 0 0.21" rpy="0 0 0"/>
             <geometry>
-                <box size="0.62 0.41 0.4"/>
+                <box size="0.75 0.45 0.42"/>
             </geometry>
             <material name="grey">
@@ -45,7 +45,7 @@
         </visual>
         <collision>
-            <origin xyz="0 0 0.2" rpy="0 0 0"/>
+            <origin xyz="0 0 0.21" rpy="0 0 0"/>
             <geometry>
-                <box size="0.62 0.41 0.4"/>
+                <box size="0.75 0.45 0.42"/>
             </geometry>
         </collision>
@@ -64,5 +64,5 @@
       <parent link="enclosure" />
       <child link = "${arm_prefix}base_link" />
-      <origin xyz="0 0 0.4" rpy="0 0 ${pi}" />
+      <origin xyz="-0.0775 0 0.42" rpy="0 0 ${pi}" />
     </joint>
   </xacro:macro>
